Commit message: Imported upstream version '0.0.2' of 'upstream'

File: widowx_arm_description/urdf/widowx.urdf.xacro (robot description, xacro)
@@ -9,5 +9,5 @@
       <child link="ph_base_link" />
    </joint-->
-   <xacro:macro name="widowx_arm" params="prefix">
+   <xacro:macro name="widowx_arm" params="parent prefix *origin">
       <!-- links -->
       <link name="${prefix}arm_base_link">
@@ -194,10 +194,9 @@
       </link>
       <!-- joints -->
-      <!--joint name="${prefix}arm_base_joint" type="fixed">
-         <origin xyz="${M_SCALE*14.5} ${M_SCALE*0.2} ${M_SCALE*0.2}" rpy="${M_PI*0} ${M_PI*0} ${-M_PI/2}" />
-         <parent link="plate_top_link" />
+      <joint name="${prefix}arm_base_joint" type="fixed">
+         <insert_block name="origin" />
+         <parent link="${parent}" />
          <child link="${prefix}arm_base_link"/>
-         <axis xyz="0 1 0" />
-      </joint-->
+      </joint>
       <joint name="${prefix}joint_1" type="revolute">
          <origin xyz="0 0 ${M_SCALE*125}" rpy="0 0 0" />
